File: PTP_Jan_Znamenacek_Project1.kicad_pcb (KiCad board)
At the start: 2 copper layers, 45 parts, among them J1 Screw_Terminal_01x02, U1 LM2574N-5, U2 74LS47, U3 4027, U4 4027, U5 HDSP-7401, U6 74LVC1G11, U7 NE555P

Commit message: PCB Crtanje
Parts:
- moved R15 17.1 mm to (170.0, 112.2), turned to -90 degrees
- moved R16 3.58 mm to (174.9, 101.2)
- moved R14 2.67 mm to (174.9, 98.0)
- moved C1 0.63 mm to (113.8, 89.2)
- moved U3 0.17 mm to (129.8, 87.6)
Routing:
- net +5V: track 0.00 -> 297.6 mm, vias 0 -> 2
- net Q1: track 0.00 -> 84.8 mm, vias 0 -> 6
- net Q0: track 0.00 -> 75.0 mm, vias 0 -> 2
- net GND: track 0.00 -> 73.4 mm
- net Q3: track 0.00 -> 63.0 mm, vias 0 -> 2
- net Reset: track 0.00 -> 61.0 mm
- net Net-(U2-b): track 0.00 -> 50.6 mm
- net Net-(U4A-J): track 0.00 -> 48.3 mm, vias 0 -> 2
- net Clock: track 0.00 -> 47.2 mm
- net Net-(U2-c): track 0.00 -> 40.3 mm
- net Q2: track 0.00 -> 37.3 mm
- net Net-(U2-a): track 0.00 -> 36.6 mm
- net Net-(U4B-J): track 0.00 -> 26.7 mm, vias 0 -> 2
- net VD: track 0.00 -> 25.7 mm
- net Net-(U2-BI): track 0.00 -> 24.8 mm, vias 0 -> 2
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- added copper zone on B.Cu, net GND

Commit message: Gerberi
Parts:
- moved R17 0.48 mm to (174.9, 91.0)
- moved R5 0.42 mm to (193.8, 90.2)
- moved R9 0.37 mm to (135.7, 83.3)
Routing:
- net +5V: track 297.6 -> 300.1 mm
Other:
- board outline added: 100 x 80 mm
- board text added: "PTP BCD Counter Jan Znamenaček"
